Commit message: Add lidar sensor, recolor chassis, and parameterize sim world
Add a 2D lidar to the robot description: lidar.xacro defines the
laser_frame link and a gazebo_ros_ray_sensor plugin publishing
sensor_msgs/LaserScan on /scan, included from robot.urdf.xacro.

Recolor the chassis from orange to gray. Dropping the material
entirely was tried first, but RViz falls back to a built-in red
for links with no <material>, so the color has to be explicit.
The Gazebo override is removed so Gazebo uses its default grey.

Add a 'world' argument to rsp_sim.launch.py naming a file in
mybot_gazebo/worlds (default empty.world), so the sim can run
against obstacles.world without editing the launch file.

Co-Authored-By: Claude Opus 5 <noreply@anthropic.com>

File: ros2_ws/src/mybot_description/description/robot.urdf.xacro (robot description, xacro)
@@ -9,3 +9,4 @@
       <xacro:include filename="gazebo_control.xacro" />
    </xacro:if>
+   <xacro:include filename="lidar.xacro" />
 </robot>

File: ros2_ws/src/mybot_description/description/robot_core.xacro (robot description, xacro)
@@ -13,4 +13,10 @@
     <material name="black">
         <color rgba="0 0 0 1" />
+    </material>
+    <material name="red">
+        <color rgba="1 0 0 1" />
+    </material>
+    <material name="gray">
+        <color rgba="0.7 0.7 0.7 1" />
     </material>
     <!-- BASE LINK -->
@@ -29,5 +35,5 @@
                 <box size="0.3 0.3 0.15" />
             </geometry>
-            <material name="orange" />
+            <material name="gray" />
         </visual>
         <collision>
@@ -41,7 +47,4 @@
         </xacro:inertial_box>
     </link>
-    <gazebo reference="chassis">
-        <material>Gazebo/Orange</material>
-    </gazebo>
     <!-- LEFT WHEEL LINK -->
     <joint name="left_wheel_joint" type="continuous">
