Commit message: Port the remaining packages to Jazzy
mybot_detection was the only package building under Jazzy. These are the
four things standing between the rest of the workspace and a clean
`colcon build` on noble.

mybot_gazebo now carries a COLCON_IGNORE, tracked rather than local.
gazebo_ros and gazebo_ros_pkgs have no Jazzy release at all --
gazebo_ros_pkgs was discontinued after Iron -- so `rosdep install
--from-paths src` fails hard on unresolved keys on every machine, not
just arm64. The .gitignore comment claiming this is per-machine was
written when the Pi was the only box that could not build the package;
that stopped being true when the workstation port also stalled.

serial_motor_demo imports serial and tkinter without declaring either.
The old Humble box had pyserial from somewhere else, which hid it; a
fresh container gets ModuleNotFoundError at `ros2 run`.

rplidar_ros was relying on <limits> and <cstring> arriving transitively
through rclcpp.hpp. GCC 13/14 pruned those, so name them. Also raise the
CMake floor to 3.16 (4.0 hard-errors on <3.5 compat), set CXX_STANDARD
17 explicitly -- 14 only worked because rclcpp::rclcpp carries
cxx_std_17 in its interface and CMake takes the max -- and drop the
ament_export_dependencies(std_msgs) for a package that is neither
declared nor found.

The Gazebo Classic sensor plugins in lidar.xacro and camera.xacro now
sit behind use_sim, alongside gazebo_control. Note the gate is inside
each file, around the <gazebo> block only: these files also define
laser_frame, camera_link and camera_link_optical, which the real robot
needs. Gating the includes themselves would have quietly removed those
frames from the hardware URDF.

example_gazebo.xacro was dead -- never included by robot.urdf.xacro,
only by a commented-out line in itself.

Co-Authored-By: Claude Opus 5 (1M context) <noreply@anthropic.com>
Claude-Session: https://claude.ai/code/session_011znZm2djb8qK4qJ2DgtBb7

File: ros2_ws/src/mybot/description/camera.xacro (robot description, xacro)
@@ -20,26 +20,33 @@
     </joint>
     <link name="camera_link_optical"></link>
-    <gazebo reference="camera_link">
-        <material>Gazebo/Red</material>
-        <sensor name="camera" type="camera">
-            <pose> 0 0 0 0 0 0 </pose>
-            <visualize>true</visualize>
-            <update_rate>10</update_rate>
-            <camera>
-                <horizontal_fov>1.089</horizontal_fov>
-                <image>
-                    <width>640</width>
-                    <height>480</height>
-                    <format>R8G8B8</format>
-                </image>
-                <clip>
-                    <near>0.05</near>
-                    <far>8.0</far>
-                </clip>
-            </camera>
-            <plugin name="camera_controller" filename="libgazebo_ros_camera.so">
-                <frame_name>camera_link_optical</frame_name>
-            </plugin>
-        </sensor>
-    </gazebo>
+    <!-- Simulation only. The links and joints above are the real robot's
+         and must always be built: rsp.launch.py needs laser_frame and
+         camera_link_optical on hardware. Only this Gazebo Classic block is
+         gated, so every Classic reference sits behind use_sim and the
+         Harmonic port is one visible job. -->
+    <xacro:if value="$(arg use_sim)">
+        <gazebo reference="camera_link">
+            <material>Gazebo/Red</material>
+            <sensor name="camera" type="camera">
+                <pose> 0 0 0 0 0 0 </pose>
+                <visualize>true</visualize>
+                <update_rate>10</update_rate>
+                <camera>
+                    <horizontal_fov>1.089</horizontal_fov>
+                    <image>
+                        <width>640</width>
+                        <height>480</height>
+                        <format>R8G8B8</format>
+                    </image>
+                    <clip>
+                        <near>0.05</near>
+                        <far>8.0</far>
+                    </clip>
+                </camera>
+                <plugin name="camera_controller" filename="libgazebo_ros_camera.so">
+                    <frame_name>camera_link_optical</frame_name>
+                </plugin>
+            </sensor>
+        </gazebo>
+    </xacro:if>
 </robot>

File: ros2_ws/src/mybot/description/lidar.xacro (robot description, xacro)
@@ -23,31 +23,38 @@
         </xacro:inertial_cylinder>
     </link>
-    <gazebo reference="laser_frame">
-        <material>Gazebo/Red</material>
-        <sensor name="laser" type="ray">
-            <pose> 0 0 0 0 0 0 </pose>
-            <visualize>false</visualize>
-            <update_rate>10</update_rate>
-            <ray>
-                <scan>
-                    <horizontal>
-                        <samples>500</samples>
-                        <min_angle>-3.14</min_angle>
-                        <max_angle>3.14</max_angle>
-                    </horizontal>
-                </scan>
-                <range>
-                    <min>0.05</min>
-                    <max>12</max>
-                </range>
-            </ray>
-            <plugin name="laser_controller" filename="libgazebo_ros_ray_sensor.so">
-                <ros>
-                    <argument>~/out:=scan</argument>
-                </ros>
-                <output_type>sensor_msgs/LaserScan</output_type>
-                <frame_name>laser_frame</frame_name>
-            </plugin>
-        </sensor>
-    </gazebo>
+    <!-- Simulation only. The links and joints above are the real robot's
+         and must always be built: rsp.launch.py needs laser_frame and
+         camera_link_optical on hardware. Only this Gazebo Classic block is
+         gated, so every Classic reference sits behind use_sim and the
+         Harmonic port is one visible job. -->
+    <xacro:if value="$(arg use_sim)">
+        <gazebo reference="laser_frame">
+            <material>Gazebo/Red</material>
+            <sensor name="laser" type="ray">
+                <pose> 0 0 0 0 0 0 </pose>
+                <visualize>false</visualize>
+                <update_rate>10</update_rate>
+                <ray>
+                    <scan>
+                        <horizontal>
+                            <samples>500</samples>
+                            <min_angle>-3.14</min_angle>
+                            <max_angle>3.14</max_angle>
+                        </horizontal>
+                    </scan>
+                    <range>
+                        <min>0.05</min>
+                        <max>12</max>
+                    </range>
+                </ray>
+                <plugin name="laser_controller" filename="libgazebo_ros_ray_sensor.so">
+                    <ros>
+                        <argument>~/out:=scan</argument>
+                    </ros>
+                    <output_type>sensor_msgs/LaserScan</output_type>
+                    <frame_name>laser_frame</frame_name>
+                </plugin>
+            </sensor>
+        </gazebo>
+    </xacro:if>
 </robot>
