Commit message: Port the simulation to Gazebo Harmonic
Finishes Phase 3 of the Jazzy runbook, the piece 0c02545 deferred. That commit
made the workspace build on Jazzy by switching simulation OFF -- a tracked
COLCON_IGNORE in mybot_gazebo -- and fencing the Classic plugin XML behind
use_sim so the port would be one visible job. This is that job.

The three plugin swaps were the easy part. What actually bites:

wheel_diameter -> wheel_radius. Harmonic's DiffDrive takes a radius. Leave the
Classic element in and gz ignores it and falls back to its DEFAULT radius of
0.2 m, so the robot drives four times too fast with four times wrong odometry
and no warning anywhere. Verified the other way: commanding 0.2 m/s reads back
as 0.2 on /odom.

max_wheel_torque has no equivalent -- gz-sim 8 DiffDrive issues a velocity
command the solver satisfies directly. max_wheel_acceleration becomes a
body-level max_linear_acceleration.

publish_wheel_tf has no equivalent either. Its job is now JointStatePublisher
plus a /joint_states bridge entry. Miss it and TF stays complete and the robot
still drives -- the wheels just never turn in RViz.

The Gazebo/Blue material blocks in robot_core.xacro are DELETED, not converted.
sdformat's URDF parser turns <material>Gazebo/Blue</material> into a <script>
that REPLACES the <ambient>/<diffuse> it already generated from the URDF
<material name="blue">. ogre2 has no Ogre material scripts, so converting them
gives white wheels -- strictly worse than having no <gazebo> block. Deleting
lets the URDF colour render. The caster's mu1/mu2 stays, in element form:
without it the caster grips and the robot will not turn. Incidentally 0c02545's
claim that "every Classic reference sits behind use_sim" was not true -- these
three blocks were ungated and landed in the real robot's URDF.

gz_frame_id is required, not cosmetic. sdformat lumps fixed joints into their
parent, so the sensors' default frame_id is a mangled
laser_frame_fixed_joint_lump__laser and RViz has no such frame. gz sdf -p warns
that gz_frame_id is "not defined in SDF"; that warning is expected and
gz-sensors reads it anyway. Confirmed at runtime: /scan arrives as laser_frame
and both camera topics as camera_link_optical.

obstacles.world was rebuilt, not converted. Its 646 lines were a GUI save: a
109-line <state> snapshot, a <gui> camera pose, every mesh inlined twice, and
empty <surface>/<self_collide> boilerplate. The signal was nine poses and two
mesh URIs pointing at Classic's model database. 163 lines now, nine Fuel
includes, obstacles static because the original gave the barrels mass 500 for
the same reason. They come out native size: <include> has no scale override and
the Classic cones carried scale 10.

Both worlds now declare Physics, UserCommands, SceneBroadcaster and Sensors
explicitly. gz-sim loads its default plugin set only if the file declares no
<plugin> at all, and each omission fails silently -- no Sensors is no /scan and
no camera at all.

Also fixes a pre-existing bug the sim launch exposed: drive_bot.rviz and
view_bot.rviz subscribed to the latched /robot_description with Volatile
durability, so whether the model appeared was a race. mybot/config/robot.rviz
already had this right.

Verified in ros2-sim-dev:0.3.0: clean colcon build of all six packages, robot
spawns, all eight bridged topics present, /scan and camera at ~10 Hz, TF one
connected tree rooted at odom, obstacles.sdf loads all nine Fuel models and the
lidar returns 94 of 500 beams at 1.68 m nearest. The real robot's URDF is
unchanged apart from the caster block and still carries laser_frame and
camera_link_optical.

Note ros2 topic hz reports nothing for the sensor topics even while they
publish normally; count with an rclpy subscriber instead. And <update_rate> on
JointStatePublisher is ignored by the gz-sim 8.11.0 Jazzy ships -- the feature
postdates it -- so /joint_states runs at the 1000 Hz physics step for now.

Co-Authored-By: Claude Opus 5 (1M context) <noreply@anthropic.com>
Claude-Session: https://claude.ai/code/session_019VoQwSSga9xATUHedevTWb

File: ros2_ws/src/mybot/description/camera.xacro (robot description, xacro)
@@ -22,14 +22,28 @@
     <!-- Simulation only. The links and joints above are the real robot's
          and must always be built: rsp.launch.py needs laser_frame and
-         camera_link_optical on hardware. Only this Gazebo Classic block is
-         gated, so every Classic reference sits behind use_sim and the
-         Harmonic port is one visible job. -->
+         camera_link_optical on hardware. Only this block is gated. -->
     <xacro:if value="$(arg use_sim)">
         <gazebo reference="camera_link">
-            <material>Gazebo/Red</material>
             <sensor name="camera" type="camera">
-                <pose> 0 0 0 0 0 0 </pose>
+                <pose>0 0 0 0 0 0</pose>
+                <update_rate>10</update_rate>
+                <always_on>true</always_on>
                 <visualize>true</visualize>
-                <update_rate>10</update_rate>
+                <!-- gz derives the info topic by replacing the last element of
+                     <topic>, so /camera/image_raw gives /camera/camera_info for
+                     free (CameraSensor::AdvertiseInfo).
+                     <gz_frame_id> replaces Classic's plugin <frame_name>. Do
+                     NOT also set <camera><optical_frame_id>: it defaults to
+                     this value, so setting both is only a way to get them out
+                     of sync.
+                     camera_link_optical, not camera_link: a gz camera looks
+                     down its link's +X, ROS optical convention is +Z forward,
+                     and camera_optical_joint above is exactly that rotation.
+                     An image rotated 90 degrees in RViz means this changed. -->
+                <topic>/camera/image_raw</topic>
+                <gz_frame_id>camera_link_optical</gz_frame_id>
+                <!-- 640x480 matches the real C920's usb_cam config in
+                     mybot_detection, so the detector could be pointed at the
+                     simulation without re-tuning. -->
                 <camera>
                     <horizontal_fov>1.089</horizontal_fov>
@@ -44,7 +58,4 @@
                     </clip>
                 </camera>
-                <plugin name="camera_controller" filename="libgazebo_ros_camera.so">
-                    <frame_name>camera_link_optical</frame_name>
-                </plugin>
             </sensor>
         </gazebo>

File: ros2_ws/src/mybot/description/gazebo_control.xacro (robot description, xacro)
@@ -1,22 +1,70 @@
 <?xml version="1.0"?>
 <robot xmlns:xacro="http://www.ros.org/wiki/xacro" name="robot">
-    <gazebo>
-        <plugin name="diff_drive" filename="libgazebo_ros_diff_drive.so">
-            <!-- The left and right wheels are the names of the joints in the URDF -->
-            <left_joint>left_wheel_joint</left_joint>
-            <right_joint>right_wheel_joint</right_joint>
-            <!-- The wheel separation is the distance between the wheels in meters -->
-            <wheel_separation>0.35</wheel_separation>
-            <wheel_diameter>0.1</wheel_diameter>
-            <!-- Limits -->
-            <max_wheel_torque>200</max_wheel_torque>
-            <max_wheel_acceleration>10.0</max_wheel_acceleration>
-            <!-- Output -->
-            <odometry_frame>odom</odometry_frame>
-            <robot_base_frame>base_link</robot_base_frame>
-            <publish_odom>true</publish_odom>
-            <publish_odom_tf>true</publish_odom_tf>
-            <publish_wheel_tf>true</publish_wheel_tf>
-        </plugin>
-    </gazebo>
+    <!-- Simulation only. Gated internally, matching lidar.xacro and
+         camera.xacro - robot.urdf.xacro also wraps the include, which is
+         belt and braces rather than the only guard. -->
+    <xacro:if value="$(arg use_sim)">
+        <gazebo>
+            <plugin filename="gz-sim-diff-drive-system"
+                    name="gz::sim::systems::DiffDrive">
+                <!-- The left and right wheels are the names of the joints in the URDF -->
+                <left_joint>left_wheel_joint</left_joint>
+                <right_joint>right_wheel_joint</right_joint>
+                <!-- Harmonic takes a RADIUS. Classic took <wheel_diameter>0.1</>.
+                     Getting this wrong is silent and expensive: gz ignores an
+                     unknown <wheel_diameter> and falls back to its DEFAULT
+                     wheel_radius of 0.2 m, so the robot drives four times too
+                     fast with four times wrong odometry and no warning. -->
+                <wheel_separation>0.35</wheel_separation>
+                <wheel_radius>0.05</wheel_radius>
+                <!-- Limits. gz-sim 8 DiffDrive has no torque limit at all: it
+                     drives the joints with a velocity command that the physics
+                     engine satisfies directly, so Classic's
+                     <max_wheel_torque>200</> has no equivalent and is dropped.
+                     Acceleration becomes a BODY-level limit rather than a
+                     per-wheel one - Classic's 10 rad/s^2 at r=0.05 is
+                     0.5 m/s^2, which is what these numbers mean. -->
+                <max_linear_acceleration>0.5</max_linear_acceleration>
+                <max_angular_acceleration>3.0</max_angular_acceleration>
+                <!-- Output. Every one of these is required. The defaults are
+                     model-scoped - /model/my_bot/cmd_vel, .../odometry,
+                     .../tf, frame_id "my_bot/odom", child_frame_id
+                     "my_bot/base_link" - which match neither the real robot's
+                     topic names nor the RViz configs. -->
+                <topic>/cmd_vel</topic>
+                <odom_topic>/odom</odom_topic>
+                <tf_topic>/tf</tf_topic>
+                <frame_id>odom</frame_id>
+                <child_frame_id>base_link</child_frame_id>
+                <odom_publish_frequency>30</odom_publish_frequency>
+            </plugin>
+            <!-- Replaces Classic's <publish_wheel_tf>true</publish_wheel_tf>,
+                 which has no Harmonic equivalent. gz publishes joint positions
+                 and the bridge carries them to /joint_states, so
+                 robot_state_publisher computes the wheel TF exactly as it does
+                 on the real robot.
+                 Without this the failure is easy to miss: TF is still complete
+                 and the robot still drives, the wheels just sit frozen at zero
+                 in RViz. -->
+            <plugin filename="gz-sim-joint-state-publisher-system"
+                    name="gz::sim::systems::JointStatePublisher">
+                <topic>/joint_states</topic>
+                <!-- IGNORED BY gz-sim 8.11.0, which is what Jazzy ships.
+                     JointStatePublisher gained <update_rate> after that release
+                     (the string is not even present in
+                     libgz-sim8-joint-state-publisher-system.so.8.11.0), so
+                     today this plugin publishes every physics step: 1000 Hz
+                     against the 1 ms step size. Left in place because it is the
+                     correct configuration and starts working on the next gz
+                     bump, but do not expect it to do anything yet - if you are
+                     wondering why /joint_states is at 1 kHz, this is why.
+                     Harmless in practice on a workstation: the message carries
+                     two joints, and /tf stays at 50 Hz. It would be worth
+                     caring about if this ever ran on the Pi. -->
+                <update_rate>30</update_rate>
+                <joint_name>left_wheel_joint</joint_name>
+                <joint_name>right_wheel_joint</joint_name>
+            </plugin>
+        </gazebo>
+    </xacro:if>
 </robot>

File: ros2_ws/src/mybot/description/lidar.xacro (robot description, xacro)
@@ -25,34 +25,51 @@
     <!-- Simulation only. The links and joints above are the real robot's
          and must always be built: rsp.launch.py needs laser_frame and
-         camera_link_optical on hardware. Only this Gazebo Classic block is
-         gated, so every Classic reference sits behind use_sim and the
-         Harmonic port is one visible job. -->
+         camera_link_optical on hardware. Only this block is gated. -->
     <xacro:if value="$(arg use_sim)">
         <gazebo reference="laser_frame">
-            <material>Gazebo/Red</material>
-            <sensor name="laser" type="ray">
-                <pose> 0 0 0 0 0 0 </pose>
+            <sensor name="laser" type="gpu_lidar">
+                <pose>0 0 0 0 0 0</pose>
+                <update_rate>10</update_rate>
+                <always_on>true</always_on>
                 <visualize>false</visualize>
-                <update_rate>10</update_rate>
-                <ray>
+                <!-- Both of these are load-bearing, and both fail silently.
+                     Without <topic>, gz publishes on the scoped path
+                     /world/default/model/my_bot/link/base_link/sensor/laser/scan
+                     - base_link, not laser_frame, because sdformat lumps
+                     fixed-joint children into their parent. Without
+                     <gz_frame_id>, header.frame_id is the sensor's mangled
+                     post-lump name (laser_frame_fixed_joint_lump__laser), and
+                     RViz has no such frame so it draws nothing. -->
+                <topic>/scan</topic>
+                <gz_frame_id>laser_frame</gz_frame_id>
+                <!-- Harmonic renames the container element <ray> -> <lidar>.
+                     sdformat still accepts <ray> as a deprecated alias, but it
+                     warns, and the deprecated path is not the one to be on. -->
+                <lidar>
                     <scan>
                         <horizontal>
                             <samples>500</samples>
+                            <!-- A multiplier on samples, not an angular step. -->
+                            <resolution>1</resolution>
                             <min_angle>-3.14</min_angle>
                             <max_angle>3.14</max_angle>
                         </horizontal>
+                        <!-- Spec-optional, included deliberately: it states the
+                             single-ring intent, and an unspecified vertical
+                             block has repeatedly been the cause of an empty
+                             scan in gz-sensors. -->
+                        <vertical>
+                            <samples>1</samples>
+                            <resolution>1</resolution>
+                            <min_angle>0</min_angle>
+                            <max_angle>0</max_angle>
+                        </vertical>
                     </scan>
                     <range>
                         <min>0.05</min>
-                        <max>12</max>
+                        <max>12.0</max>
+                        <resolution>0.01</resolution>
                     </range>
-                </ray>
-                <plugin name="laser_controller" filename="libgazebo_ros_ray_sensor.so">
-                    <ros>
-                        <argument>~/out:=scan</argument>
-                    </ros>
-                    <output_type>sensor_msgs/LaserScan</output_type>
-                    <frame_name>laser_frame</frame_name>
-                </plugin>
+                </lidar>
             </sensor>
         </gazebo>

File: ros2_ws/src/mybot/description/robot.urdf.xacro (robot description, xacro)
@@ -1,7 +1,12 @@
 <?xml version="1.0"?>
 <robot xmlns:xacro="http://www.ros.org/wiki/xacro"  name="robot">
-   <!-- Gazebo plugin tags are inert outside simulation, but the Pi has no
-        Gazebo at all, so keep them out of the real robot's URDF.
-        mybot_gazebo's launch file passes use_sim:=true. -->
+   <!-- Gazebo plugin tags are inert outside simulation - URDF parsers ignore
+        <gazebo> - but there is no reason to ship the simulator's plugins and
+        sensors in the real robot's description, so they are gated.
+        mybot_gazebo's launch file passes use_sim:=true.
+        Note this is no longer "the Pi cannot run Gazebo": ros_gz IS published
+        for arm64 on Jazzy. It is deliberately not installed in the Pi's image,
+        because running a simulator on the robot is a bad use of a Pi 5.
+        See .devcontainer/RUNBOOK-jazzy-upgrade.md. -->
    <xacro:arg name="use_sim" default="false"/>
    <xacro:include filename="robot_core.xacro" />

File: ros2_ws/src/mybot/description/robot_core.xacro (robot description, xacro)
@@ -70,7 +70,4 @@
         </xacro:inertial_cylinder>
     </link>
-    <gazebo reference="left_wheel">
-        <material>Gazebo/Blue</material>
-    </gazebo>
     <!-- RIGHT WHEEL LINK -->
     <joint name="right_wheel_joint" type="continuous">
@@ -96,7 +93,4 @@
         </xacro:inertial_cylinder>
     </link>
-    <gazebo reference="right_wheel">
-        <material>Gazebo/Blue</material>
-    </gazebo>
     <!-- CASTER WHEEL LINK -->
     <joint name="caster_wheel_joint" type="fixed">
@@ -121,8 +115,18 @@
         </xacro:inertial_sphere>
     </link>
+    <!-- Low friction so the caster slides instead of dragging; without it the
+         robot will not turn. sdformat's URDF parser maps these onto the link's
+         collision as <surface><friction><ode><mu>/<mu2>, which gz-physics'
+         DART plugin reads. Unlike a <material> child, this survives the move
+         to Harmonic unchanged.
+         Ungated on purpose. This block is inert outside simulation - URDF
+         parsers ignore <gazebo> - and gating it would mean the description
+         differed between the two machines for no gain. The Classic material
+         children that used to sit alongside it are gone: Gazebo/* are Ogre
+         material SCRIPTS, which ogre2 does not have, and sdformat lets them
+         overwrite the colours the URDF <material> elements already produce. -->
     <gazebo reference="caster_wheel">
-        <material>Gazebo/Black</material>
-        <mu1 value="0.001" />
-        <mu2 value="0.001" />
+        <mu1>0.001</mu1>
+        <mu2>0.001</mu2>
     </gazebo>
 </robot>
